Commit message: Added LiDAR module to URDF robot description

File: steer_bot_description/urdf/steer_bot.urdf.xacro (robot description, xacro)
@@ -134,7 +134,63 @@
     <origin xyz="${-base_length/2+axle_offset} ${+base_width/2+axle_offset} 0" rpy="${-90 * deg_to_rad} 0 0"/>
   </xacro:rear_wheel_lr>
+  <link name="lidar">
+    <inertial>
+      <origin xyz="0 0 0.15" rpy="0 0 0"/>
+      <mass value="1"/>
+      <inertia ixx="100"  ixy="0"  ixz="0" iyy="100" iyz="0" izz="100" />
+    </inertial>
+    <visual>
+      <origin xyz="0 0 0.15" rpy="0 0 0"/>
+      <geometry>
+        <cylinder length="0.055" radius="0.0508"/>
+      </geometry>
+      <material name="red"/>
+    </visual>
+    <collision>
+      <origin xyz="0 0 0.15" rpy="0 0 0"/>
+      <geometry>
+        <cylinder length="0.055" radius="0.0508"/>
+      </geometry>
+    </collision>
+    </link>
+    <joint name="lidar_joint" type="fixed">
+      <parent link = "base_link"/>
+      <child link = "lidar"/>
+      <pose>-0.032 0 0.171 0 0 0</pose>
+      <axis>
+        <xyz>0 0 1</xyz>
+        <use_parent_model_frame>true</use_parent_model_frame>
+      </axis>
+    </joint>
   <!-- Colour -->
   <gazebo reference="base_link">
     <material>Gazebo/Green</material>
   </gazebo>
+  <gazebo reference="lidar">
+    <material>Gazebo/Red</material>
+    <sensor name="laser" type="ray">
+        <pose> 0 0 0 0 0 0 </pose>
+        <visualize>true</visualize>
+        <update_rate>10</update_rate>
+        <ray>
+          <scan>
+              <horizontal>
+                  <samples>360</samples>
+                  <min_angle>-3.14</min_angle>
+                  <max_angle>3.14</max_angle>
+              </horizontal>
+          </scan>
+          <range>
+              <min>0.3</min>
+              <max>12</max>
+          </range>
+        </ray>
+        <!--laser_controller libgazebo_ros_ray_sensor.so!-->
+        <plugin name="ros_ray_sensor_controller" filename="libgazebo_ros_laser.so">
+            <output_type>sensor_msgs/LaserScan</output_type>
+            <frameName>lidar</frameName>
+            <topicName>/scan</topicName>
+        </plugin>
+    </sensor>
+  </gazebo>
 </robot>

Commit message: Update URDF
- Put camera on its own link
- Refined robot cosmetic appearance
Issues:
Camera and Lidar are in the middle of the robot, technically on the base link. This is not ideal for accurate simulation of the robot.

File: steer_bot_description/urdf/steer_bot.urdf.xacro (robot description, xacro)
@@ -61,8 +61,8 @@
       </geometry>
     </collision>
-    <xacro:solid_cuboid_inertial
+    <!--<xacro:solid_cuboid_inertial
         rpy="0 0 0" xyz="0 0 0"
         mass="${base_mass}"
-        x="${base_length}" y="${base_width}" z="${base_height}" />
+        x="${base_length}" y="${base_width}" z="${base_height}" />-->
   </link>
   <!-- Front steer and rear wheel joints required for ackermann_steering_controller -->
@@ -145,5 +145,5 @@
         <cylinder length="0.055" radius="0.0508"/>
       </geometry>
-      <material name="red"/>
+      <!--<material name="red"/>-->
     </visual>
     <collision>
@@ -153,4 +153,24 @@
       </geometry>
     </collision>
+    </link>
+    <link name="camera">
+      <inertial>
+        <origin xyz="0.2 0 0.1" rpy="0 0 0"/>
+        <mass value="0.25"/>
+        <inertia ixx="100"  ixy="0"  ixz="0" iyy="100" iyz="0" izz="100" />
+      </inertial>
+      <visual>
+        <origin xyz="0.2 0 0.1" rpy="0 0 0"/>
+        <geometry>
+          <box size="${steer_radius} ${steer_radius} ${steer_thickness}"/>
+        </geometry>
+        <!--<material name="red"/>-->
+      </visual>
+      <collision>
+        <origin xyz="0.2 0 0.1" rpy="0 0 0"/>
+        <geometry>
+          <box size="${steer_radius} ${steer_radius} ${steer_thickness}"/>
+        </geometry>
+      </collision>
     </link>
     <joint name="lidar_joint" type="fixed">
@@ -160,15 +180,36 @@
       <axis>
         <xyz>0 0 1</xyz>
+        <use_parent_model_frame>false</use_parent_model_frame>
+      </axis>
+      <limit effort="${steer_effort}"
+             lower="0" upper="0"
+             velocity="${steer_velocity}"/>
+    </joint>
+    <joint name="camera_joint" type="fixed">
+      <parent link = "base_link"/>
+      <child link = "camera"/>
+      <pose>0.2 0 0.171 0 0 0</pose>
+      <axis>
+        <xyz>0 0 1</xyz>
         <use_parent_model_frame>true</use_parent_model_frame>
       </axis>
+      <!--<limit effort="${steer_effort}"
+             lower="0" upper="0"
+             velocity="${steer_velocity}"/>-->
     </joint>
   <!-- Colour -->
   <gazebo reference="base_link">
-    <material>Gazebo/Green</material>
+    <material>Gazebo/Grey</material>
   </gazebo>
   <gazebo reference="lidar">
-    <material>Gazebo/Red</material>
+    <material>Gazebo/RedGlow</material>
     <sensor name="laser" type="ray">
-        <pose> 0 0 0 0 0 0 </pose>
+        <parent link="lidar"/>
+        <origin xyz="0 0 0" rpy="0 0 0"/>
+        <pose> 0 0 0.1 0 0 0 </pose>
+        <axis>
+          <xyz>0 0 1</xyz>
+          <use_parent_model_frame>true</use_parent_model_frame>
+        </axis>
         <visualize>true</visualize>
         <update_rate>10</update_rate>
@@ -194,6 +235,13 @@
     </sensor>
   </gazebo>
-  <gazebo reference="front_steer_link">
+  <gazebo reference="camera">
+    <material>Gazebo/BlueGlow</material>
     <sensor type="camera" name="camera1">
+      <!--<origin xyz="0.25 0 0.1" rpy="0 0 0"/>-->
+      <pose> 0.25 0 0.3 0 0 0 </pose>
+      <!--<axis>
+          <xyz>0 0 1</xyz>
+          <use_parent_model_frame>true</use_parent_model_frame>
+      </axis>-->
       <visualize>true</visualize>
       <update_rate>30.0</update_rate>
@@ -206,5 +254,5 @@
         </image>
         <clip>
-          <near>0.02</near>
+          <near>1</near>
           <far>300</far>
         </clip>
@@ -220,6 +268,6 @@
         <imageTopicName>/camera1/image_raw</imageTopicName>
         <cameraInfoTopicName>/camera1/camera_info</cameraInfoTopicName>
-        <frameName>front_steer_link</frameName>
-        <hackBaseline>0.07</hackBaseline>
+        <frameName>camera</frameName>
+        <hackBaseline>0.2</hackBaseline>
         <distortionK1>0.0</distortionK1>
         <distortionK2>0.0</distortionK2>

File: steer_bot_description/urdf/wheel.xacro (robot description, xacro)
@@ -162,5 +162,5 @@
     </gazebo>
     <gazebo reference="${name}_wheel_link">
-      <material>Gazebo/Red</material>
+      <material>Gazebo/Black</material>
     </gazebo>
   </xacro:macro>
@@ -299,5 +299,5 @@
     </transmission>
     <gazebo reference="${name}_wheel_link">
-      <material>Gazebo/Red</material>
+      <material>Gazebo/Black</material>
     </gazebo>
   </xacro:macro>

Commit message: Sensors now mounted in correct places on robot + got meshes for them
also changed the lidar to perform like the TiM-P lidar we are getting

File: steer_bot_description/urdf/steer_bot.urdf.xacro (robot description, xacro)
@@ -17,4 +17,6 @@
   <!-- Include xacro for inertials, materials and wheels -->
   <xacro:include filename="$(find steer_bot_description)/urdf/wheel.xacro"/>
+  <xacro:include filename="$(find steer_bot_description)/urdf/SICK_lidar.xacro"/>
+  <xacro:include filename="$(find steer_bot_description)/urdf/kinect_cam.xacro"/>
   <xacro:property name="robot_namespace" value="/steer_bot"/>
   <!-- Gazebo plugins -->
@@ -31,11 +33,11 @@
   <xacro:property name="deg_to_rad" value="0.01745329251994329577"/>
   <!-- Robot base dimensions -->
-  <xacro:property name="base_length" value="0.5" />
-  <xacro:property name="base_width" value="0.3" />
-  <xacro:property name="base_height" value="0.1" />
+  <xacro:property name="base_length" value="0.38735" /> <!--fake 0.5 real 0.139-->
+  <xacro:property name="base_width" value="0.23495" /> <!--fake 0.3 real 0.139-->
+  <xacro:property name="base_height" value="0.06985" /> <!--fake 0.1 real 0.139-->
   <xacro:property name="base_mass" value="5" />
   <!-- Wheel link dimensions -->
-  <xacro:property name="wheel_radius" value="0.1" />
-  <xacro:property name="wheel_thickness" value="0.08" />
+  <xacro:property name="wheel_radius" value="0.0635" /> <!--fake 0.1 real 0.139-->
+  <xacro:property name="wheel_thickness" value="0.0381" /> <!--fake 0.08 real 0.139-->
   <xacro:property name="wheel_mass" value="1" />
   <!-- Steering link dimensions -->
@@ -44,6 +46,6 @@
   <xacro:property name="steer_mass" value="1" />
   <!-- Axle positions -->
-  <xacro:property name="axle_offset" value="0.05" />
-  <xacro:property name="steer_offset" value="0.02" />
+  <xacro:property name="axle_offset" value="0.0254" /> <!--fake 0.05 real 0.139-->
+  <xacro:property name="steer_offset" value="0.0254" /> <!--fake 0.02 real 0.139-->
   <!-- Base link -->
   <link name="base_link">
@@ -134,67 +136,37 @@
     <origin xyz="${-base_length/2+axle_offset} ${+base_width/2+axle_offset} 0" rpy="${-90 * deg_to_rad} 0 0"/>
   </xacro:rear_wheel_lr>
-  <link name="lidar">
-    <inertial>
-      <origin xyz="0 0 0.15" rpy="0 0 0"/>
-      <mass value="1"/>
-      <inertia ixx="100"  ixy="0"  ixz="0" iyy="100" iyz="0" izz="100" />
-    </inertial>
-    <visual>
-      <origin xyz="0 0 0.15" rpy="0 0 0"/>
-      <geometry>
-        <cylinder length="0.055" radius="0.0508"/>
-      </geometry>
-      <!--<material name="red"/>-->
-    </visual>
-    <collision>
-      <origin xyz="0 0 0.15" rpy="0 0 0"/>
-      <geometry>
-        <cylinder length="0.055" radius="0.0508"/>
-      </geometry>
-    </collision>
-    </link>
+    <xacro:SICK_lidar name="lidar">
+      <origin xyz="0 0 0" rpy="0 0 0"/>
+    </xacro:SICK_lidar>
+    <xacro:kinect_cam name="camera_real">
+      <origin xyz="0 0 0" rpy="0 0 0"/>
+    </xacro:kinect_cam>
     <link name="camera">
       <inertial>
-        <origin xyz="0.2 0 0.1" rpy="0 0 0"/>
+        <origin xyz="0 0 0" rpy="0 0 0"/>
         <mass value="0.25"/>
         <inertia ixx="100"  ixy="0"  ixz="0" iyy="100" iyz="0" izz="100" />
       </inertial>
       <visual>
-        <origin xyz="0.2 0 0.1" rpy="0 0 0"/>
+        <origin xyz="0 0 0" rpy="0 0 0"/>
         <geometry>
-          <box size="${steer_radius} ${steer_radius} ${steer_thickness}"/>
+          <box size="0.01 0.01 0.01"/>
         </geometry>
-        <!--<material name="red"/>-->
       </visual>
       <collision>
-        <origin xyz="0.2 0 0.1" rpy="0 0 0"/>
+        <origin xyz="0 0 0" rpy="0 0 0"/>
         <geometry>
-          <box size="${steer_radius} ${steer_radius} ${steer_thickness}"/>
+          <box size="0.01 0.01 0.01"/>
         </geometry>
       </collision>
     </link>
-    <joint name="lidar_joint" type="fixed">
-      <parent link = "base_link"/>
-      <child link = "lidar"/>
-      <pose>-0.032 0 0.171 0 0 0</pose>
-      <axis>
-        <xyz>0 0 1</xyz>
-        <use_parent_model_frame>false</use_parent_model_frame>
-      </axis>
-      <limit effort="${steer_effort}"
-             lower="0" upper="0"
-             velocity="${steer_velocity}"/>
-    </joint>
     <joint name="camera_joint" type="fixed">
       <parent link = "base_link"/>
       <child link = "camera"/>
-      <pose>0.2 0 0.171 0 0 0</pose>
+      <pose>0 0 0 0 0 0</pose>
       <axis>
         <xyz>0 0 1</xyz>
         <use_parent_model_frame>true</use_parent_model_frame>
       </axis>
-      <!--<limit effort="${steer_effort}"
-             lower="0" upper="0"
-             velocity="${steer_velocity}"/>-->
     </joint>
   <!-- Colour -->
@@ -202,47 +174,9 @@
     <material>Gazebo/Grey</material>
   </gazebo>
-  <gazebo reference="lidar">
-    <material>Gazebo/RedGlow</material>
-    <sensor name="laser" type="ray">
-        <parent link="lidar"/>
-        <origin xyz="0 0 0" rpy="0 0 0"/>
-        <pose> 0 0 0.1 0 0 0 </pose>
-        <axis>
-          <xyz>0 0 1</xyz>
-          <use_parent_model_frame>true</use_parent_model_frame>
-        </axis>
-        <visualize>true</visualize>
-        <update_rate>10</update_rate>
-        <ray>
-          <scan>
-              <horizontal>
-                  <samples>360</samples>
-                  <min_angle>-3.14</min_angle>
-                  <max_angle>3.14</max_angle>
-              </horizontal>
-          </scan>
-          <range>
-              <min>0.3</min>
-              <max>12</max>
-          </range>
-        </ray>
-        <!--laser_controller libgazebo_ros_ray_sensor.so!-->
-        <plugin name="ros_ray_sensor_controller" filename="libgazebo_ros_laser.so">
-            <output_type>sensor_msgs/LaserScan</output_type>
-            <frameName>lidar</frameName>
-            <topicName>/scan</topicName>
-        </plugin>
-    </sensor>
-  </gazebo>
   <gazebo reference="camera">
-    <material>Gazebo/BlueGlow</material>
-    <sensor type="camera" name="camera1">
-      <!--<origin xyz="0.25 0 0.1" rpy="0 0 0"/>-->
+    <material>Gazebo/Black</material>
+    <sensor type="camera" name="cameraFake">
       <pose> 0.25 0 0.3 0 0 0 </pose>
-      <!--<axis>
-          <xyz>0 0 1</xyz>
-          <use_parent_model_frame>true</use_parent_model_frame>
-      </axis>-->
-      <visualize>true</visualize>
+      <visualize>false</visualize>
       <update_rate>30.0</update_rate>
       <camera>
@@ -266,6 +200,6 @@
         <alwaysOn>true</alwaysOn>
         <updateRate>30.0</updateRate>
-        <imageTopicName>/camera1/image_raw</imageTopicName>
-        <cameraInfoTopicName>/camera1/camera_info</cameraInfoTopicName>
+        <imageTopicName>/camera2/image_raw</imageTopicName>
+        <cameraInfoTopicName>/camera2/camera_info</cameraInfoTopicName>
         <frameName>camera</frameName>
         <hackBaseline>0.2</hackBaseline>
