Commit message: making sure steer_bot urdf is functioning correctly

File: steer_bot_description/urdf/bicycle_bot.urdf.xacro (robot description, xacro)
@@ -32,5 +32,5 @@
             front_wheel_joint
         </jointName>
-        <updateRate>50</updateRate>
+        <updateRate>20</updateRate>
         <alwaysOn>true</alwaysOn>
     </plugin>

File: steer_bot_description/urdf/kinect_cam.xacro (robot description, xacro)
@@ -38,5 +38,5 @@
         <material>Gazebo/Black</material>
         <sensor type="camera" name="camera1">
-        <origin xyz="0.25 0 0.1" rpy="0 0 0"/>
+        <origin xyz="0 0 0" rpy="0 0 0"/>
         <pose> 0.2 0 0.1 0 0 0 </pose>
         <!--<axis>
@@ -49,11 +49,11 @@
             <horizontal_fov>1.3962634</horizontal_fov>
             <image>
-            <width>800</width>
-            <height>800</height>
+            <width>640</width>
+            <height>480</height>
             <format>R8G8B8</format>
             </image>
             <clip>
             <near>1</near>
-            <far>300</far>
+            <far>50</far>
             </clip>
             <noise>
@@ -68,5 +68,5 @@
             <imageTopicName>/camera1/image_raw</imageTopicName>
             <cameraInfoTopicName>/camera1/camera_info</cameraInfoTopicName>
-            <frameName>camera</frameName>
+            <frameName>camera_real</frameName>
             <hackBaseline>0.2</hackBaseline>
             <distortionK1>0.0</distortionK1>

File: steer_bot_description/urdf/steer_bot.urdf.xacro (robot description, xacro)
@@ -145,6 +145,6 @@
       <inertial>
         <origin xyz="0 0 0" rpy="0 0 0"/>
-        <mass value="0.25"/>
-        <inertia ixx="100"  ixy="0"  ixz="0" iyy="100" iyz="0" izz="100" />
+        <mass value="0.01"/>
+        <inertia ixx="0"  ixy="0"  ixz="0" iyy="0" iyz="0" izz="0" />
       </inertial>
       <visual>
@@ -199,5 +199,5 @@
       <plugin name="camera2_camera_controller" filename="libgazebo_ros_camera.so">
         <alwaysOn>true</alwaysOn>
-        <updateRate>30.0</updateRate>
+        <updateRate>15.0</updateRate>
         <imageTopicName>/camera2/image_raw</imageTopicName>
         <cameraInfoTopicName>/camera2/camera_info</cameraInfoTopicName>
