Commit message: fixed mesh file locations

File: steer_bot_description/urdf/SICK_lidar.xacro (robot description, xacro)
@@ -9,5 +9,5 @@
             <origin xyz="0 0 0.15" rpy="0 0 0"/>
             <mass value="1"/>
-            <inertia ixx="100"  ixy="0"  ixz="0" iyy="100" iyz="0" izz="100" />
+            <inertia ixx="0"  ixy="0"  ixz="0" iyy="0" iyz="0" izz="0" />
         </inertial>
         <visual>
@@ -38,12 +38,12 @@
         <sensor name="laser" type="ray">
             <parent link="${name}"/>
-            <origin xyz="0 0 0.15" rpy="0 0 0"/>
+            <!--<origin xyz="0 0 0.15" rpy="0 0 0"/>-->
             <pose> 0 0 0.15 0 0 0 </pose>
             <axis>
-            <xyz>0 0 1</xyz>
-            <use_parent_model_frame>true</use_parent_model_frame>
+                <xyz>0 0 1</xyz>
+                <use_parent_model_frame>true</use_parent_model_frame>
             </axis>
             <visualize>true</visualize>
-            <update_rate>10</update_rate>
+            <update_rate>15</update_rate>
             <ray>
             <scan>
@@ -55,5 +55,5 @@
             </scan>
             <range>
-                <min>0.3</min>
+                <min>0.1</min>
                 <max>25</max>
             </range>

File: steer_bot_description/urdf/kinect_cam.xacro (robot description, xacro)
@@ -9,5 +9,5 @@
         <origin xyz="0.2 0 0.1" rpy="0 0 0"/>
         <mass value="0.25"/>
-        <inertia ixx="100"  ixy="0"  ixz="0" iyy="100" iyz="0" izz="100" />
+        <inertia ixx="0"  ixy="0"  ixz="0" iyy="0" iyz="0" izz="0" />
       </inertial>
       <visual>
@@ -19,7 +19,8 @@
       </visual>
       <collision>
-        <origin xyz="0.2 0 0.1" rpy="0 0 0"/>
+        <origin xyz="0 0 0" rpy="0 0 0"/>
         <geometry>
-          <mesh filename="package://steer_bot_description/meshes/kinect_v2.stl" scale="0.01 0.01 0.01"/>
+          <box size="0.01 0.01 0.01"/>
+          <!--<mesh filename="package://steer_bot_description/meshes/kinect_v2.stl" scale="0.01 0.01 0.01"/>-->
         </geometry>
       </collision>
@@ -44,5 +45,5 @@
         </axis>-->
         <visualize>true</visualize>
-        <update_rate>30.0</update_rate>
+        <update_rate>15.0</update_rate>
         <camera>
             <horizontal_fov>1.3962634</horizontal_fov>
@@ -64,5 +65,5 @@
         <plugin name="camera1_camera_controller" filename="libgazebo_ros_camera.so">
             <alwaysOn>true</alwaysOn>
-            <updateRate>30.0</updateRate>
+            <updateRate>15.0</updateRate>
             <imageTopicName>/camera1/image_raw</imageTopicName>
             <cameraInfoTopicName>/camera1/camera_info</cameraInfoTopicName>

Commit message: Fixed collision meshes

File: steer_bot_description/urdf/SICK_lidar.xacro (robot description, xacro)
@@ -21,5 +21,5 @@
             <origin xyz="0 0 0.15" rpy="0 0 0"/>
             <geometry>
-                <mesh filename="package://zm_robot_description/meshes/sick_tim_5xx.stl"/>
+                <mesh filename="package://steer_bot_description/meshes/sick_tim_5xx.stl"/>
             </geometry>
         </collision>

File: steer_bot_description/urdf/kinect_cam.xacro (robot description, xacro)
@@ -14,5 +14,5 @@
         <origin xyz="0.2 0 0.1" rpy="0 0 0"/>
         <geometry>
-          <mesh filename="package://zm_robot_description/meshes/kinect_v2.stl" scale="0.01 0.01 0.01"/>
+          <mesh filename="package://steer_bot_description/meshes/kinect_v2.stl" scale="0.01 0.01 0.01"/>
         </geometry>
         <!--<material name="red"/>-->

Commit message: Spring Break Update #1
- Fixes wheelbase length (L), was 0.38735 now 0.315

File: steer_bot_description/urdf/SICK_lidar.xacro (robot description, xacro)
@@ -44,5 +44,5 @@
                 <use_parent_model_frame>true</use_parent_model_frame>
             </axis>
-            <visualize>true</visualize>
+            <visualize>false</visualize>
             <update_rate>15</update_rate>
             <ray>

File: steer_bot_description/urdf/kinect_cam.xacro (robot description, xacro)
@@ -44,5 +44,5 @@
             <use_parent_model_frame>true</use_parent_model_frame>
         </axis>-->
-        <visualize>true</visualize>
+        <visualize>false</visualize>
         <update_rate>15.0</update_rate>
         <camera>

File: steer_bot_description/urdf/steer_bot.urdf.xacro (robot description, xacro)
@@ -46,5 +46,5 @@
   <xacro:property name="steer_mass" value="1" />
   <!-- Axle positions -->
-  <xacro:property name="axle_offset" value="0.0254" /> <!--fake 0.05 real 0.139-->
+  <xacro:property name="axle_offset" value="0.036175" /> <!--fake 0.05 real 0.035-->
   <xacro:property name="steer_offset" value="0.0254" /> <!--fake 0.02 real 0.139-->
   <!-- Base link -->
